File: docs/indication_schematic/indication_schematic.kicad_sch (KiCad schematic)
At the start: 7 parts, among them J1 Conn_01x04_MountingPin, J2 Conn_01x03_MountingPin, J3 Conn_01x03_MountingPin, U1 PTN78000H_EUS-5, U2 PTN78000H_EUS-5, U3 PTN78000H_EUS-5

Commit message: Finished Indication Schematic
Parts:
- added J4: Conn_02x08_Top_Bottom, symbol Connector_Generic:Conn_02x08_Top_Bottom
- added J5: Conn_01x06, symbol Connector_Generic:Conn_01x06
Connections:
- net GND: now also A1.29 (GND), A1.6 (GND), J4.7 (Pin_7), J5.3 (Pin_3)
- net B: now reaches A1.10 (A1)
- net B: now also J4.4 (Pin_4)
- net C: now reaches A1.11 (A2)
- net C: now also J4.11 (Pin_11)
- net D: now reaches A1.12 (A3)
- net D: now also J4.3 (Pin_3)
- net TXD: now reaches A1.15 (D0/RX)
- net TXD: now also J5.4 (Pin_4)
- net RXD: now reaches A1.16 (D1/TX)
- net RXD: now also J5.5 (Pin_5)
- net R1: now reaches A1.17 (D2)
- net R1: now also J4.16 (Pin_16)
- net G1: now reaches A1.18 (D3)
- net G1: now also J4.8 (Pin_8)
- net B1: now reaches A1.19 (D4)
- net B1: now also J4.15 (Pin_15)
- net R2: now reaches A1.20 (D5)
- net R2: now also J4.14 (Pin_14)
- net G2: now reaches A1.21 (D6)
- net G2: now also J4.6 (Pin_6)
- net B2: now reaches A1.22 (D7)
- net B2: now also J4.13 (Pin_13)
- net CLK: now reaches A1.23 (D8)
- net CLK: now also J4.10 (Pin_10)
- net OE: now reaches A1.24 (D9)
- net OE: now also J4.9 (Pin_9)
- net LAT: now reaches A1.25 (D10)
- net LAT: now also J4.2 (Pin_2)
- net VCC: now reaches A1.5 (+5V)
- net VCC: now also J5.2 (Pin_2)
- net A: now reaches A1.9 (A0)
- net A: now also J4.12 (Pin_12)
- new net: J2.1 (Pin_1), J3.1 (Pin_1), U2.5 (VO)
- new net: A1.26 (D11), J2.2 (Pin_2)
- new net: A1.27 (D12), J3.2 (Pin_2)
- new net EN: J5.1 (Pin_1)
- new net STATE: J5.6 (Pin_6)
Other:
- note added: "DC-DC Step-down Buck Converter"
- note added: "HC-02 Bluetooth Connector"
- note added: "Matrix Data Connector"
- moved on the sheet: J2, J3
